Commit message: Integration with cameras

File: openarm_description/urdf/ee/openarm_hand_arguments.xacro (robot description, xacro)
@@ -12,5 +12,5 @@
   <xacro:arg name="tcp_rpy" default="0 0 0" />
   <!-- Is the robot being simulated in gazebo? -->
-  <!-- <xacro:arg name="gazebo" default="false" /> -->
+  <xacro:arg name="gazebo" default="false" />
   <!-- Name of the description package -->
   <xacro:arg name="description_pkg" default="openarm_description" />

File: openarm_description/urdf/robot/openarm_robot.xacro (robot description, xacro)
@@ -40,4 +40,5 @@
             >
     <xacro:include filename="$(find openarm_description)/urdf/body/openarm_neck.xacro" />
+    <xacro:include filename="$(find openarm_description)/urdf/sensors/camera.xacro"/>
     <xacro:include filename="$(find openarm_description)/urdf/arm/openarm_macro.xacro" />
     <xacro:include filename="$(find openarm_description)/urdf/arm/openarm_arm.xacro" />
@@ -65,6 +66,14 @@
         kinematics="${body_kinematics}"
         kinematics_link="${body_kinematics_link}" />
-	<!-- neck -->
-	<xacro:openarm_neck parent="openarm_body_link0" />
+        <!-- neck -->
+        <xacro:openarm_neck parent="openarm_body_link0" />
+        <!-- 1. LEFT ARM END-EFFECTOR CAMERA -->
+        <xacro:openarm_camera name="left_ee_camera" parent_link="openarm_left_hand_tcp">
+            <origin xyz="0.03 0 0" rpy="0 0 0"/>
+        </xacro:openarm_camera>
+        <!-- 2. RIGHT ARM END-EFFECTOR CAMERA -->
+        <xacro:openarm_camera name="right_ee_camera" parent_link="openarm_right_hand_tcp">
+            <origin xyz="0.03 0 0" rpy="0 0 0"/>
+        </xacro:openarm_camera>
         <!-- left arm -->
         <xacro:openarm_arm
